Commit message: update

File: src/bookle_calib/bookle_description/urdf/bookle.xacro (robot description, xacro)
@@ -70,128 +70,68 @@
 	</link>
 	<link name="left_frame">
-		<pose>0 -0.1 .1 0 0 0</pose>
+		<origin xyz="0 -0.1 0.1" rpy="0 0 0" />
 		<collision name="left_collision">
-			<pose>0 .0075 -0.03 0 0 0</pose>
+			<origin xyz="0 0.0075 -0.03" rpy="0 0 0" />
 			<geometry>
-				<box>
-					<size>.08 .002 .06</size>
-				</box>
+				<box size=".08 .002 .06" />
 			</geometry>
-			<surface>
-				<friction>
-					<ode>
-						<mu>0.3</mu>
-						<mu2>0.3</mu2>
-						<slip1>1.0</slip1>
-						<slip2>1.0</slip2>
-					</ode>
-				</friction>
-			</surface>
 		</collision>
 		<visual name="left_visual">
-			<pose>0 .0075 -0.03 0 0 0</pose>
+			<origin xyz="0 .0075 -0.03" rpy="0 0 0" />
 			<geometry>
-				<box>
-					<size>.08 .002 .06</size>
-				</box>
+				<box size=".08 .002 .06" />
 			</geometry>
 		</visual>
 		<collision name="right_collision">
-			<pose>0 -0.0075 -0.03 0 0 0</pose>
+			<origin xya="0 -0.0075 -0.03" rpy="0 0 0"/>
 			<geometry>
-				<box>
-					<size>.08 .002 .06</size>
-				</box>
+				<box size=".08 .002 .06" />
 			</geometry>
-			<surface>
-				<friction>
-					<ode>
-						<mu>0.3</mu>
-						<mu2>0.3</mu2>
-						<slip1>1.0</slip1>
-						<slip2>1.0</slip2>
-					</ode>
-				</friction>
-			</surface>
 		</collision>
 		<visual name="right_visual">
-			<pose>0 -0.0075 -0.03 0 0 0</pose>
+			<origin xyz="0 -0.0075 -0.03" rpy="0 0 0" />
 			<geometry>
-				<box>
-					<size>.08 .002 .06</size>
-				</box>
+				<box size=".08 .002 .06" />
 			</geometry>
 		</visual>
 	</link>
 	<link name="right_frame">
-		<pose>0 0.1 .1 0 0 0</pose>
+		<origin xyz="0 0.1 0.1" rpy="0 0 0" />
 		<collision name="left_collision">
-			<pose>0 .0075 -0.03 0 0 0</pose>
+			<origin xyz="0 .0075 -0.03" rpy="0 0 0" />
 			<geometry>
-				<box>
-					<size>.08 .002 .06</size>
-				</box>
+				<box size=".08 .002 .06" />
 			</geometry>
-			<surface>
-				<friction>
-					<ode>
-						<mu>0.3</mu>
-						<mu2>0.3</mu2>
-						<slip1>1.0</slip1>
-						<slip2>1.0</slip2>
-					</ode>
-				</friction>
-			</surface>
 		</collision>
 		<visual name="left_visual">
-			<pose>0 .0075 -0.03 0 0 0</pose>
+			<origin xyz="0 .0075 -0.03" rpy="0 0 0" />
 			<geometry>
-				<box>
-					<size>.08 .002 .06</size>
-				</box>
+				<box size=".08 .002 .06" />
 			</geometry>
 		</visual>
 		<collision name="right_collision">
-			<pose>0 -0.0075 -0.03 0 0 0</pose>
+			<origin xyz="0 -0.0075 -0.03" rpy="0 0 0" />
 			<geometry>
-				<box>
-					<size>.08 .002 .06</size>
-				</box>
+				<box size=".08 .002 .06" />
 			</geometry>
-			<surface>
-				<friction>
-					<ode>
-						<mu>0.3</mu>
-						<mu2>0.3</mu2>
-						<slip1>1.0</slip1>
-						<slip2>1.0</slip2>
-					</ode>
-				</friction>
-			</surface>
 		</collision>
 		<visual name="right_visual">
-			<pose>0 -0.0075 -0.03 0 0 0</pose>
+			<origin xyz="0 -0.0075 -0.03" rpy="0 0 0" />
 			<geometry>
-				<box>
-					<size>.08 .002 .06</size>
-				</box>
+				<box size=".08 .002 .06" />
 			</geometry>
 		</visual>
 	</link>
 	<joint type="revolute" name="left_wheel_hinge">
-		<pose>0 .1 .04 0 0 0</pose>
-		<child>left_wheel</child>
-		<parent>left_frame</parent>
-		<axis>
-			<xyz>0 1 0</xyz>
-		</axis>
+		<origin xyz="0 .1 .04" rpy="0 0 0" />
+		<child link="left_wheel" />
+		<parent link="left_frame" />
+		<axis xyz="0 1 0" />
 	</joint>
 	<joint type="revolute" name="right_wheel_hinge">
-		<pose>0 -0.1 .04 0 0 0</pose>
-		<child>right_wheel</child>
-		<parent>right_frame</parent>
-		<axis>
-			<xyz>0 1 0</xyz>
-		</axis>
+		<origin xyz="0 -0.1 .04" rpy="0 0 0" />
+		<child link="right_wheel" />
+		<parent link="right_frame" />
+		<axis xyz="0 1 0" />
 	</joint>
 	<include>
