Commit message: udpate

File: bookle_description/urdf/bookle.xacro (robot description, xacro)
@@ -190,23 +190,3 @@
 		</inertial>
 	</link>
-	<transmission name="tran1">
-		<type>transmission_interface/SimpleTransmission</type>
-		<joint name="joint1">
-			<hardwareInterface>EffortJointInterface</hardwareInterface>
-		</joint>
-		<actuator name="motor1">
-			<hardwareInterface>EffortJointInterface</hardwareInterface>
-			<mechanicalReduction>1</mechanicalReduction>
-		</actuator>
-	</transmission>
-	<transmission name="tran2">
-		<type>transmission_interface/SimpleTransmission</type>
-		<joint name="joint2">
-			<hardwareInterface>EffortJointInterface</hardwareInterface>
-		</joint>
-		<actuator name="motor2">
-			<hardwareInterface>EffortJointInterface</hardwareInterface>
-			<mechanicalReduction>1</mechanicalReduction>
-		</actuator>
-	</transmission>
 </robot>

Commit message: update

File: bookle_description/urdf/bookle.xacro (robot description, xacro)
@@ -7,5 +7,5 @@
 	<link name="chassis">
 		<collision name="collision">
-			<origin xyz="0 0 .1" rpy="0 0 0" />
+			<origin xyz="0 0 0.1" rpy="0 0 0" />
 			<geometry>
 				<cylinder radius="0.15" length="0.003" />
@@ -13,5 +13,5 @@
 		</collision>
 		<visual name="visual">
-			<origin xyz="0 0 .1" rpy="0 0 0" />
+			<origin xyz="0 0 0.1" rpy="0 0 0" />
 			<geometry>
 				<cylinder radius="0.15" length="0.003" />
@@ -19,5 +19,5 @@
 		</visual>
 		<collision name="front_caster_collision">
-			<origin xyz="0.1 0 -0.05" rpy="0 1.5707 1.5707" />
+			<origin xyz="0.1 0 0.05" rpy="0 1.5707 1.5707" />
 			<geometry>
 				<cylinder radius="0.05" length="0.015" />
@@ -25,5 +25,5 @@
 		</collision>
 		<visual name="front_caster_visual">
-			<origin xyz="0.1 0 -0.05" rpy="0 1.5707 1.5707" />
+			<origin xyz="0.1 0 0.05" rpy="0 1.5707 1.5707" />
 			<geometry>
 				<cylinder radius="0.05" length="0.015" />
@@ -31,5 +31,5 @@
 		</visual>
 		<collision name="back_caster_collision">
-			<origin xyz="-0.1 0 -0.05" rpy="0 1.5707 1.5707" />
+			<origin xyz="-0.1 0 0.05" rpy="0 1.5707 1.5707" />
 			<geometry>
 				<cylinder radius="0.05" length="0.015" />
@@ -37,5 +37,5 @@
 		</collision>
 		<visual name="back_caster_visual">
-			<origin xyz="-0.1 0 -0.05" rpy="0 1.5707 1.5707" />
+			<origin xyz="-0.1 0 0.05" rpy="0 1.5707 1.5707" />
 			<geometry>
 				<cylinder radius="0.05" length="0.015" />
@@ -44,6 +44,6 @@
 	</link>
 	<link name="left_wheel">
-		<origin xyz="0 .1 .04" rpy="0 1.5707 1.5707" />
 		<collision name="collision">
+			<origin xyz="0 0 0" rpy="0 1.5707 1.5707" />
 			<geometry>
 				<cylinder radius="0.04" length="0.015" />
@@ -51,12 +51,18 @@
 		</collision>
 		<visual name="visual">
-			<geometry>
-				<cylinder radius="0.04" length="0.015" />
-			</geometry>
-		</visual>
+			<origin xyz="0 0 0" rpy="0 1.5707 1.5707" />
+			<geometry>
+				<cylinder radius="0.04" length="0.015" />
+			</geometry>
+		</visual>
+		<inertial>
+			<mass value="1" />
+			<origin xyz="0 0 1" rpy="0 0 0"/>
+			<inertia ixx="1" ixy="0" ixz="0" iyy="1" iyz="0" izz="1" />
+		</inertial>
 	</link>
 	<link name="right_wheel">
-		<origin xyz="0 -0.1 .04" rpy="0 1.5707 1.5707" />
 		<collision name="collision">
+			<origin xyz="0 0 0" rpy="0 1.5707 1.5707" />
 			<geometry>
 				<cylinder radius="0.04" length="0.015" />
@@ -64,13 +70,19 @@
 		</collision>
 		<visual name="visual">
-			<geometry>
-				<cylinder radius="0.04" length="0.015" />
-			</geometry>
-		</visual>
+			<origin xyz="0 0 0" rpy="0 1.5707 1.5707" />
+			<geometry>
+				<cylinder radius="0.04" length="0.015" />
+			</geometry>
+		</visual>
+		<inertial>
+			<mass value="1" />
+			<origin xyz="0 0 1" rpy="0 0 0"/>
+			<inertia ixx="1" ixy="0" ixz="0" iyy="1" iyz="0" izz="1" />
+		</inertial>
 	</link>
 	<link name="left_frame">
-		<origin xyz="0 -0.1 0.1" rpy="0 0 0" />
+		<!-- <origin xyz="0 -0.1 0.1" rpy="0 0 0" /> -->
 		<collision name="left_collision">
-			<origin xyz="0 0.0075 -0.03" rpy="0 0 0" />
+			<origin xyz="0 0.0075 0" rpy="0 0 0" />
 			<geometry>
 				<box size=".08 .002 .06" />
@@ -78,5 +90,5 @@
 		</collision>
 		<visual name="left_visual">
-			<origin xyz="0 .0075 -0.03" rpy="0 0 0" />
+			<origin xyz="0 0.0075 0" rpy="0 0 0" />
 			<geometry>
 				<box size=".08 .002 .06" />
@@ -84,5 +96,5 @@
 		</visual>
 		<collision name="right_collision">
-			<origin xya="0 -0.0075 -0.03" rpy="0 0 0"/>
+			<origin xya="0 -0.0075 0" rpy="0 0 0"/>
 			<geometry>
 				<box size=".08 .002 .06" />
@@ -90,5 +102,5 @@
 		</collision>
 		<visual name="right_visual">
-			<origin xyz="0 -0.0075 -0.03" rpy="0 0 0" />
+			<origin xyz="0 -0.0075 0" rpy="0 0 0" />
 			<geometry>
 				<box size=".08 .002 .06" />
@@ -97,7 +109,7 @@
 	</link>
 	<link name="right_frame">
-		<origin xyz="0 0.1 0.1" rpy="0 0 0" />
+		<!-- <origin xyz="0 0.1 0.1" rpy="0 0 0" /> -->
 		<collision name="left_collision">
-			<origin xyz="0 .0075 -0.03" rpy="0 0 0" />
+			<origin xyz="0 .0075 0" rpy="0 0 0" />
 			<geometry>
 				<box size=".08 .002 .06" />
@@ -105,5 +117,5 @@
 		</collision>
 		<visual name="left_visual">
-			<origin xyz="0 .0075 -0.03" rpy="0 0 0" />
+			<origin xyz="0 .0075 0" rpy="0 0 0" />
 			<geometry>
 				<box size=".08 .002 .06" />
@@ -111,5 +123,5 @@
 		</visual>
 		<collision name="right_collision">
-			<origin xyz="0 -0.0075 -0.03" rpy="0 0 0" />
+			<origin xyz="0 -0.0075 0" rpy="0 0 0" />
 			<geometry>
 				<box size=".08 .002 .06" />
@@ -117,5 +129,5 @@
 		</collision>
 		<visual name="right_visual">
-			<origin xyz="0 -0.0075 -0.03" rpy="0 0 0" />
+			<origin xyz="0 -0.0075 0" rpy="0 0 0" />
 			<geometry>
 				<box size=".08 .002 .06" />
@@ -124,5 +136,5 @@
 	</link>
 	<joint type="revolute" name="left_wheel_hinge">
-		<origin xyz="0 .1 .04" rpy="0 0 0" />
+		<origin xyz="0 0 -0.03" rpy="0 0 0" />
 		<child link="left_wheel" />
 		<parent link="left_frame" />
@@ -131,5 +143,5 @@
 	</joint>
 	<joint type="revolute" name="right_wheel_hinge">
-		<origin xyz="0 -0.1 .04" rpy="0 0 0" />
+		<origin xyz="0 0 -0.03" rpy="0 0 0" />
 		<child link="right_wheel" />
 		<parent link="right_frame" />
@@ -138,5 +150,5 @@
 	</joint>
 	<joint type="fixed" name="left_frame_joint">
-		<origin xyz="0 -0.1 0.1" rpy="0 0 0" />
+		<origin xyz="0 0.1 0.069" rpy="0 0 0" />
 		<child link="left_frame" />
 		<parent link="chassis" />
@@ -144,5 +156,5 @@
 	</joint>
 	<joint type="fixed" name="right_frame_joint">
-		<origin xyz="0 0.1 0.1" rpy="0 0 0" />
+		<origin xyz="0 -0.1 0.069" rpy="0 0 0" />
 		<child link="right_frame" />
 		<parent link="chassis" />

Commit message: run

File: bookle_description/urdf/bookle.xacro (robot description, xacro)
@@ -42,4 +42,9 @@
 			</geometry>
 		</visual>
+		<inertial>
+			<origin xyz="0 0 .1" rpy="0 0 0" />
+			<mass value="1" />
+			<inertia ixx="1.0" ixy="0.0" ixz="0.0" iyy="1.0" iyz="0.0" izz="1.0" />
+		</inertial>
 	</link>
 	<link name="left_wheel">
@@ -58,5 +63,5 @@
 		<inertial>
 			<mass value="1" />
-			<origin xyz="0 0 1" rpy="0 0 0"/>
+			<origin xyz="0 0 0" rpy="0 0 0"/>
 			<inertia ixx="1" ixy="0" ixz="0" iyy="1" iyz="0" izz="1" />
 		</inertial>
@@ -77,5 +82,5 @@
 		<inertial>
 			<mass value="1" />
-			<origin xyz="0 0 1" rpy="0 0 0"/>
+			<origin xyz="0 0 0" rpy="0 0 0"/>
 			<inertia ixx="1" ixy="0" ixz="0" iyy="1" iyz="0" izz="1" />
 		</inertial>
@@ -107,4 +112,9 @@
 			</geometry>
 		</visual>
+		<inertial>
+			<origin xyz="0 0 0" rpy="0 0 0" />
+			<mass value="1" />
+			<inertia ixx="1.0" ixy="0.0" ixz="0.0" iyy="1.0" iyz="0.0" izz="1.0" />
+		</inertial>
 	</link>
 	<link name="right_frame">
@@ -134,4 +144,9 @@
 			</geometry>
 		</visual>
+		<inertial>
+			<origin xyz="0 0 0" rpy="0 0 0" />
+			<mass value="1" />
+			<inertia ixx="1.0" ixy="0.0" ixz="0.0" iyy="1.0" iyz="0.0" izz="1.0" />
+		</inertial>
 	</link>
 	<joint type="revolute" name="left_wheel_hinge">
@@ -150,5 +165,5 @@
 	</joint>
 	<joint type="fixed" name="left_frame_joint">
-		<origin xyz="0 0.1 0.069" rpy="0 0 0" />
+		<origin xyz="0 0.1 0.07" rpy="0 0 0" />
 		<child link="left_frame" />
 		<parent link="chassis" />
@@ -156,9 +171,27 @@
 	</joint>
 	<joint type="fixed" name="right_frame_joint">
-		<origin xyz="0 -0.1 0.069" rpy="0 0 0" />
+		<origin xyz="0 -0.1 0.07" rpy="0 0 0" />
 		<child link="right_frame" />
 		<parent link="chassis" />
 		<axis xyz="1 0 0" />
 	</joint>
+	<transmission name="left_wheel_trans" type="SimpleTransmission">
+		<type>transmission_interface/SimpleTransmission</type>
+		<actuator name="left_wheel_motor">
+			<mechanicalReduction>1</mechanicalReduction>
+		</actuator>
+		<joint name="left_wheel">
+			<hardwareInterface>VelocityJointInterface</hardwareInterface>
+		</joint>
+	</transmission>
+	<transmission name="right_wheel_trans" type="SimpleTransmission">
+		<type>transmission_interface/SimpleTransmission</type>
+		<actuator name="right_wheel_motor">
+			<mechanicalReduction>1</mechanicalReduction>
+		</actuator>
+		<joint name="right_wheel">
+			<hardwareInterface>VelocityJointInterface</hardwareInterface>
+		</joint>
+	</transmission>
 	<!-- <include>
 		<uri>model://hokuyo</uri>

Commit message: update

File: bookle_description/urdf/bookle.xacro (robot description, xacro)
@@ -213,8 +213,8 @@
 		<origin xyz="0.1 0 0.135" rpy="0 0 0"/>
 		<parent link="chassis"/>
-		<child link="hokuyo_link"/>
+		<child link="velodyne"/>
 	</joint>
 	<!-- Hokuyo Laser -->
-	<link name="hokuyo_link">
+	<link name="velodyne">
 		<collision>
 			<origin xyz="0 0 0" rpy="0 0 0"/>

Commit message: update

File: bookle_description/urdf/bookle.xacro (robot description, xacro)
@@ -210,5 +210,5 @@
 	</joint> -->
 	<joint name="hokuyo_joint" type="fixed">
-		<axis xyz="0 1 0" />
+		<axis xyz="0 0 1" />
 		<origin xyz="0.1 0 0.135" rpy="0 0 0"/>
 		<parent link="chassis"/>

Commit message: add occupancy grid to gridmap

File: bookle_description/urdf/bookle.xacro (robot description, xacro)
@@ -5,5 +5,5 @@
 	<!-- Import all Gazebo-customization elements, including Gazebo colors -->
 	<xacro:include filename="$(find bookle_description)/urdf/bookle.gazebo" />
-	<link name="chassis">
+	<link name="base_link">
 		<collision name="collision">
 			<origin xyz="0 0 0.1" rpy="0 0 0" />
@@ -167,5 +167,5 @@
 		<origin xyz="0 0.1 0.07" rpy="0 0 0" />
 		<child link="left_frame" />
-		<parent link="chassis" />
+		<parent link="base_link" />
 		<axis xyz="1 0 0" />
 	</joint>
@@ -173,5 +173,5 @@
 		<origin xyz="0 -0.1 0.07" rpy="0 0 0" />
 		<child link="right_frame" />
-		<parent link="chassis" />
+		<parent link="base_link" />
 		<axis xyz="1 0 0" />
 	</joint>
@@ -200,5 +200,5 @@
 	<joint name="hokuyo_joint" type="revolute">
 		<child>hokuyo::link</child>
-		<parent>chassis</parent>
+		<parent>base_link</parent>
 		<axis>
 			<xyz>0 0 1</xyz>
@@ -212,9 +212,9 @@
 		<axis xyz="0 0 1" />
 		<origin xyz="0.1 0 0.135" rpy="0 0 0"/>
-		<parent link="chassis"/>
-		<child link="velodyne"/>
+		<parent link="base_link"/>
+		<child link="base_laser"/>
 	</joint>
 	<!-- Hokuyo Laser -->
-	<link name="velodyne">
+	<link name="base_laser">
 		<collision>
 			<origin xyz="0 0 0" rpy="0 0 0"/>

Commit message: update

File: bookle_description/urdf/bookle.xacro (robot description, xacro)
@@ -5,4 +5,18 @@
 	<!-- Import all Gazebo-customization elements, including Gazebo colors -->
 	<xacro:include filename="$(find bookle_description)/urdf/bookle.gazebo" />
+	<link name="base_footprint">
+		<collision name="base_footprint_collision">
+			<origin xyz="0 0 0"  rpy="0 0 0" />
+			<geometry>
+				<box size="0.001 0.001 0.001" />
+			</geometry>
+		</collision>
+		<visual name="base_footprint_visual">
+			<origin xyz="0 0 0" rpy="0 0 0" />
+			<geometry>
+				<box size="0.001 0.001 0.001" />
+			</geometry>
+		</visual>
+	</link>
 	<link name="base_link">
 		<collision name="collision">
@@ -87,5 +101,4 @@
 	</link>
 	<link name="left_frame">
-		<!-- <origin xyz="0 -0.1 0.1" rpy="0 0 0" /> -->
 		<collision name="left_collision">
 			<origin xyz="0 0.0075 0" rpy="0 0 0" />
@@ -119,5 +132,4 @@
 	</link>
 	<link name="right_frame">
-		<!-- <origin xyz="0 0.1 0.1" rpy="0 0 0" /> -->
 		<collision name="left_collision">
 			<origin xyz="0 .0075 0" rpy="0 0 0" />
@@ -150,17 +162,22 @@
 		</inertial>
 	</link>
-	<joint type="revolute" name="left_wheel_hinge">
+	<joint type="fixed" name="base_footprint_joint">
+		<origin xyz="0 0 0" rpy="0 0 0" />
+		<child link="base_link" />
+		<parent link="base_footprint" />
+	</joint>
+	<joint type="continuous" name="left_wheel_joint">
 		<origin xyz="0 0 -0.03" rpy="0 0 0" />
 		<child link="left_wheel" />
 		<parent link="left_frame" />
 		<axis xyz="0 1 0" />
-		<limit effort="30" velocity="0.5" lower="-3.14" upper="3.14"/>
-	</joint>
-	<joint type="revolute" name="right_wheel_hinge">
+		<!-- <limit effort="30" velocity="0.5" lower="-3.14" upper="3.14"/>  -->
+	</joint>
+	<joint type="continuous" name="right_wheel_joint">
 		<origin xyz="0 0 -0.03" rpy="0 0 0" />
 		<child link="right_wheel" />
 		<parent link="right_frame" />
 		<axis xyz="0 1 0" />
-		<limit effort="30" velocity="0.5" lower="-3.14" upper="3.14"/>
+		<!-- <limit effort="30" velocity="0.5" lower="-3.14" upper="3.14"/>  -->
 	</joint>
 	<joint type="fixed" name="left_frame_joint">
@@ -181,5 +198,5 @@
 			<mechanicalReduction>1</mechanicalReduction>
 		</actuator>
-		<joint name="left_wheel">
+		<joint name="left_wheel_joint">
 			<hardwareInterface>VelocityJointInterface</hardwareInterface>
 		</joint>
@@ -190,5 +207,5 @@
 			<mechanicalReduction>1</mechanicalReduction>
 		</actuator>
-		<joint name="right_wheel">
+		<joint name="right_wheel_joint">
 			<hardwareInterface>VelocityJointInterface</hardwareInterface>
 		</joint>

Commit message: update

File: bookle_description/urdf/bookle.xacro (robot description, xacro)
@@ -20,5 +20,5 @@
 	</link>
 	<link name="base_link">
-		<collision name="collision">
+		<collision name="base_link_collision">
 			<origin xyz="0 0 0.1" rpy="0 0 0" />
 			<geometry>
@@ -26,5 +26,5 @@
 			</geometry>
 		</collision>
-		<visual name="visual">
+		<visual name="base_link_visual">
 			<origin xyz="0 0 0.1" rpy="0 0 0" />
 			<geometry>
@@ -58,19 +58,21 @@
 		<inertial>
 			<origin xyz="0 0 .1" rpy="0 0 0" />
-			<mass value="1" />
+			<mass value="0.5" />
 			<inertia ixx="1.0" ixy="0.0" ixz="0.0" iyy="1.0" iyz="0.0" izz="1.0" />
 		</inertial>
 	</link>
 	<link name="left_wheel">
-		<collision name="collision">
-			<origin xyz="0 0 0" rpy="0 1.5707 1.5707" />
-			<geometry>
-				<cylinder radius="0.04" length="0.015" />
-			</geometry>
-		</collision>
-		<visual name="visual">
-			<origin xyz="0 0 0" rpy="0 1.5707 1.5707" />
-			<geometry>
-				<cylinder radius="0.04" length="0.015" />
+		<collision name="left_wheel_collision">
+			<origin xyz="0 0 0" rpy="0 1.5707 1.5707" />
+			<geometry>
+				<!-- <cylinder radius="0.04" length="0.015" /> -->
+				<box size="0.04 0.04 0.01" />
+			</geometry>
+		</collision>
+		<visual name="left_wheel_visual">
+			<origin xyz="0 0 0" rpy="0 1.5707 1.5707" />
+			<geometry>
+				<!-- <cylinder radius="0.04" length="0.015" /> -->
+				<box size="0.04 0.04 0.01" />
 			</geometry>
 		</visual>
@@ -82,14 +84,16 @@
 	</link>
 	<link name="right_wheel">
-		<collision name="collision">
-			<origin xyz="0 0 0" rpy="0 1.5707 1.5707" />
-			<geometry>
-				<cylinder radius="0.04" length="0.015" />
-			</geometry>
-		</collision>
-		<visual name="visual">
-			<origin xyz="0 0 0" rpy="0 1.5707 1.5707" />
-			<geometry>
-				<cylinder radius="0.04" length="0.015" />
+		<collision name="right_wheel_collision">
+			<origin xyz="0 0 0" rpy="0 1.5707 1.5707" />
+			<geometry>
+				<!-- <cylinder radius="0.04" length="0.015" /> -->
+				<box size="0.04 0.04 0.01" />
+			</geometry>
+		</collision>
+		<visual name="right_wheel_visual">
+			<origin xyz="0 0 0" rpy="0 1.5707 1.5707" />
+			<geometry>
+				<!-- <cylinder radius="0.04" length="0.015" /> -->
+				<box size="0.04 0.04 0.01" />
 			</geometry>
 		</visual>
@@ -101,5 +105,5 @@
 	</link>
 	<link name="left_frame">
-		<collision name="left_collision">
+		<collision name="left_frame1_collision">
 			<origin xyz="0 0.0075 0" rpy="0 0 0" />
 			<geometry>
@@ -107,5 +111,5 @@
 			</geometry>
 		</collision>
-		<visual name="left_visual">
+		<visual name="left_frame1_visual">
 			<origin xyz="0 0.0075 0" rpy="0 0 0" />
 			<geometry>
@@ -113,5 +117,5 @@
 			</geometry>
 		</visual>
-		<collision name="right_collision">
+		<collision name="left_frame2_collision">
 			<origin xya="0 -0.0075 0" rpy="0 0 0"/>
 			<geometry>
@@ -119,5 +123,5 @@
 			</geometry>
 		</collision>
-		<visual name="right_visual">
+		<visual name="left_frame2_visual">
 			<origin xyz="0 -0.0075 0" rpy="0 0 0" />
 			<geometry>
@@ -132,5 +136,5 @@
 	</link>
 	<link name="right_frame">
-		<collision name="left_collision">
+		<collision name="right_frame1_collision">
 			<origin xyz="0 .0075 0" rpy="0 0 0" />
 			<geometry>
@@ -138,5 +142,5 @@
 			</geometry>
 		</collision>
-		<visual name="left_visual">
+		<visual name="right_frame1_visual">
 			<origin xyz="0 .0075 0" rpy="0 0 0" />
 			<geometry>
@@ -144,5 +148,5 @@
 			</geometry>
 		</visual>
-		<collision name="right_collision">
+		<collision name="right_frame2_collision">
 			<origin xyz="0 -0.0075 0" rpy="0 0 0" />
 			<geometry>
@@ -150,5 +154,5 @@
 			</geometry>
 		</collision>
-		<visual name="right_visual">
+		<visual name="right_frame2_visual">
 			<origin xyz="0 -0.0075 0" rpy="0 0 0" />
 			<geometry>
@@ -172,4 +176,6 @@
 		<parent link="left_frame" />
 		<axis xyz="0 1 0" />
+		<dynamics damping="0.1" friction="0.1"/>
+		<limit effort="100" velocity="100"/>
 		<!-- <limit effort="30" velocity="0.5" lower="-3.14" upper="3.14"/>  -->
 	</joint>
@@ -179,4 +185,6 @@
 		<parent link="right_frame" />
 		<axis xyz="0 1 0" />
+		<dynamics damping="0.1" friction="0.2"/>
+		<limit effort="100" velocity="100"/>
 		<!-- <limit effort="30" velocity="0.5" lower="-3.14" upper="3.14"/>  -->
 	</joint>
@@ -186,4 +194,5 @@
 		<parent link="base_link" />
 		<axis xyz="1 0 0" />
+		<dynamics damping="0.1" friction="0.2"/>
 	</joint>
 	<joint type="fixed" name="right_frame_joint">
@@ -192,4 +201,5 @@
 		<parent link="base_link" />
 		<axis xyz="1 0 0" />
+		<dynamics damping="0.1" friction="0.1"/>
 	</joint>
 	<transmission name="left_wheel_trans" type="SimpleTransmission">
